File: LM399.sch (KiCad schematic (older format))
At the start: 13 parts, among them U2 LM399, U3 LT1001

Commit message: Increased footprint size of R1 from 0603 to 0805
Parts:
- R1: footprint Resistor_SMD:R_0603_1608Metric -> Resistor_SMD:R_0805_2012Metric
Changed lines of the file:
@@
 F 0 "R1" V 5693 2800 50  0000 C CNN
 F 1 "7.5K" V 5784 2800 50  0000 C CNN
-F 2 "Resistor_SMD:R_0603_1608Metric" V 5830 2800 50  0001 C CNN
+F 2 "Resistor_SMD:R_0805_2012Metric" V 5830 2800 50  0001 C CNN
 F 3 "" H 5900 2800 50  0001 C CNN
 F 4 "Welwyn" H 5900 2800 60  0001 C CNN "MFN"

Commit message: Changed trace width to 0.25 mm to make it more robust Added bypass capacitor to the temperature sensor Rotated open source logo to fit it onto the board
Parts:
- NT2, NT4, NT5: footprint Custom_footprints:NET-TIE-0.20mm -> Custom_footprints:NET-TIE-0.25mm
- NT3: footprint Custom_footprints:NET-TIE-0.15mm -> Custom_footprints:NET-TIE-0.25mm
Changed lines of the file:
@@
 EESchema Schematic File Version 4
 LIBS:reference_board-cache
-EELAYER 26 0
+EELAYER 29 0
 EELAYER END
 $Descr A4 11693 8268
@@
 F 0 "NT3" V 6854 5988 50  0000 L CNN
 F 1 "NET-TIE" V 6945 5988 50  0000 L CNN
-F 2 "Custom_footprints:NET-TIE-0.15mm" H 6900 5800 50  0001 C CNN
+F 2 "Custom_footprints:NET-TIE-0.25mm" H 6900 5800 50  0001 C CNN
 F 3 "" H 6900 5900 60  0000 C CNN
 	1    6900 5900
@@
 F 0 "NT2" V 5004 3588 50  0000 L CNN
 F 1 "NET-TIE" V 5095 3588 50  0000 L CNN
-F 2 "Custom_footprints:NET-TIE-0.20mm" H 5050 3400 50  0001 C CNN
+F 2 "Custom_footprints:NET-TIE-0.25mm" H 5050 3400 50  0001 C CNN
 F 3 "" H 5050 3500 60  0000 C CNN
 	1    5050 3500
@@
 	1    0    0    -1
 $EndComp
+Wire Wire Line
+	6900 2800 6900 3450
+Wire Wire Line
+	6900 3650 6900 4050
+Wire Wire Line
+	6900 4050 6900 4250
+Wire Wire Line
+	6900 4450 6900 4800
+Connection ~ 6900 4800
 $Comp
 L Device:Net-Tie_2 NT4
@@
 F 0 "NT4" V 6854 3638 50  0000 L CNN
 F 1 "NET-TIE" V 6945 3638 50  0000 L CNN
-F 2 "Custom_footprints:NET-TIE-0.20mm" H 6900 3450 50  0001 C CNN
+F 2 "Custom_footprints:NET-TIE-0.25mm" H 6900 3450 50  0001 C CNN
 F 3 "" H 6900 3550 60  0000 C CNN
 	1    6900 3550
 	0    1    1    0
 $EndComp
-Wire Wire Line
-	6900 2800 6900 3450
-Wire Wire Line
-	6900 3650 6900 4050
 $Comp
 L Device:Net-Tie_2 NT5
@@
 F 0 "NT5" V 6854 4438 50  0000 L CNN
 F 1 "NET-TIE" V 6945 4438 50  0000 L CNN
-F 2 "Custom_footprints:NET-TIE-0.20mm" H 6900 4250 50  0001 C CNN
+F 2 "Custom_footprints:NET-TIE-0.25mm" H 6900 4250 50  0001 C CNN
 F 3 "" H 6900 4350 60  0000 C CNN
 	1    6900 4350
 	0    1    1    0
 $EndComp
-Wire Wire Line
-	6900 4050 6900 4250
-Wire Wire Line
-	6900 4450 6900 4800
-Connection ~ 6900 4800
 $EndSCHEMATC

Commit message: Updated the LM399 footprint to match the KiCAD guidelines
Parts:
- U2: footprint Custom_footprints:LM399 -> Custom_footprints:TO-46-4_ThermalShield; symbol Linear-Technology:LM399 -> Reference_Voltage:LM399; MFN Linear Technology -> Analog Devices
Changed lines of the file:
@@
 $EndDescr
 $Comp
-L Linear-Technology:LM399 U2
+L Reference_Voltage:LM399 U2
 U 1 1 591A5398
 P 4000 3300
 F 0 "U2" H 4408 3353 60  0000 L CNN
 F 1 "LM399" H 4408 3247 60  0000 L CNN
-F 2 "Custom_footprints:LM399" H 4000 3250 60  0001 C CNN
+F 2 "Custom_footprints:TO-46-4_ThermalShield" H 4000 3250 60  0001 C CNN
 F 3 "" H 4000 3250 60  0001 C CNN
-F 4 "Linear Technology" H 4000 3300 60  0001 C CNN "MFN"
+F 4 "Analog Devices" H 4000 3300 60  0001 C CNN "MFN"
 F 5 "LM399AH" H 4000 3300 60  0001 C CNN "MFP"
 	1    4000 3300
 	1    0    0    -1
 $EndComp
-Text HLabel 3850 2400 1    60   UnSpc ~ 0
+Text HLabel 3800 2450 1    60   UnSpc ~ 0
 V-heater+
-Text HLabel 3850 3950 3    60   UnSpc ~ 0
+Text HLabel 3800 3900 3    60   UnSpc ~ 0
 V_heater-
 Text HLabel 2500 2500 1    60   UnSpc ~ 0
@@
 Text Label 6900 6100 3    60   ~ 0
 V_zener+
-Text Label 4150 2750 1    60   ~ 0
+Text Label 4200 2800 1    60   ~ 0
 V_zener+
 $Comp
@@
 	4600 2800 4600 2850
 Wire Wire Line
-	3850 2850 3850 2400
-Wire Wire Line
-	3850 3950 3850 3750
+	3800 2900 3800 2450
+Wire Wire Line
+	3800 3900 3800 3700
 Wire Wire Line
 	2500 2500 2500 2950
@@
 	5450 4150 5600 4150
 Wire Wire Line
-	4150 3950 5600 3950
+	4200 3950 5600 3950
 Wire Wire Line
 	5000 2800 5050 2800
@@
 Connection ~ 5800 4500
 Wire Wire Line
-	4150 3750 4150 3800
+	4200 3700 4200 3800
 Wire Wire Line
 	2500 2950 2800 2750
@@
 	6900 6000 6900 6100
 Wire Wire Line
-	4150 2750 4150 2850
+	4200 2800 4200 2900
 Wire Wire Line
 	5050 2800 5050 3400
@@
 	5050 3600 5050 3800
 Wire Wire Line
-	5050 3800 4150 3800
-Connection ~ 4150 3800
+	5050 3800 4200 3800
+Connection ~ 4200 3800
 Wire Wire Line
 	6900 4800 6550 4800
@@
 	5800 4500 5800 5050
 Wire Wire Line
-	4150 3800 4150 3950
+	4200 3800 4200 3950
 Wire Wire Line
 	6550 5350 6750 5350

Commit message: Updated resistor requirements (changed R1 from 5 ppm to 10 ppm) Rotated all text labels by 180° to match the main pcb Fixed soldermask to preventsolder from shorting rectangular pins to GND
Parts:
- R1: Alternative (none) -> Panasonic ERA-6ARB752V
Other:
- note added: "17k: Pin 1 -> Pin 2\nPin 1 is correctly\nmarked on the package"
- note added: "The output drift with the zener current\nis about 5 x 10^-3 ppm / ppm.\nIn order to meet the LM399 specs make sure the resistor\nhas a maximum TCR of 10 ppm / K (results in 0.06 ppm / K)."
- note added: "e.g. ERA-6ARB752V (10 ppm)\nPCF0805-13-7K5-B-T1 (5 ppm),\nTE Connectivity RU73X2A7K5LTDF (2 ppm),\nVishay S102 (2 ppm)"
- note removed: "The output drift with the zener current\nis about 5 x 10^-3 ppm / ppm.\nIn order to meet the LM399 specs make sure the resistor\nhas a maximum TCR of 5 ppm / K (results in 0.03 ppm / K)."
- note removed: "Use precision resistors\nwith an extremly low TCR\nor a network with very good\ntracking TCR."
- note removed: "e.g. PCF0805-13-7K5-B-T1 (5 ppm),\nTE Connectivity RU73X2A7K5LTDF (2 ppm),\nVishay S102 (2 ppm)\n\nPCF0805-13-3K-B-T1. (5 ppm),\nVishay S102 (2 ppm)"
- moved on the sheet: U2
Changed lines of the file:
@@
 Sheet 2 2
 Title "LM399 negative voltage reference"
-Date "2019-01-11"
-Rev "v3.1.0"
+Date "2019-06-28"
+Rev "v3.1.1"
 Comp ""
 Comment1 "Copyright (©) 2018, Patrick Baus <patrick.baus@physik.tu-darmstadt.de>"
@@
 L Reference_Voltage:LM399 U2
 U 1 1 591A5398
-P 4000 3300
-F 0 "U2" H 4408 3353 60  0000 L CNN
-F 1 "LM399" H 4408 3247 60  0000 L CNN
-F 2 "Custom_footprints:TO-46-4_ThermalShield" H 4000 3250 60  0001 C CNN
-F 3 "" H 4000 3250 60  0001 C CNN
-F 4 "Analog Devices" H 4000 3300 60  0001 C CNN "MFN"
-F 5 "LM399AH" H 4000 3300 60  0001 C CNN "MFP"
-	1    4000 3300
-	1    0    0    -1
-$EndComp
-Text HLabel 3800 2450 1    60   UnSpc ~ 0
+P 4100 3500
+AR Path="/591A5398" Ref="U2"  Part="1"
+AR Path="/591A50E3/591A5398" Ref="U2"  Part="1"
+F 0 "U2" H 4300 3550 60  0000 L CNN
+F 1 "LM399" H 4300 3450 60  0000 L CNN
+F 2 "Custom_footprints:TO-46-4_ThermalShield" H 4100 3450 60  0001 C CNN
+F 3 "" H 4100 3450 60  0001 C CNN
+F 4 "Analog Devices" H 4100 3500 60  0001 C CNN "MFN"
+F 5 "LM399AH" H 4100 3500 60  0001 C CNN "MFP"
+	1    4100 3500
+	1    0    0    -1
+$EndComp
+Text HLabel 4000 2850 1    60   UnSpc ~ 0
 V-heater+
-Text HLabel 3800 3900 3    60   UnSpc ~ 0
+Text HLabel 4000 3900 3    60   UnSpc ~ 0
 V_heater-
 Text HLabel 2500 2500 1    60   UnSpc ~ 0
 V_zener+_force
-Text Notes 8000 5750 0    60   ~ 0
-Use precision resistors\nwith an extremly low TCR\nor a network with very good\ntracking TCR.
 $Comp
 L Device:R R1
@@
 F 4 "Welwyn" H 5900 2800 60  0001 C CNN "MFN"
 F 5 "PCF0805-13-7K5-B-T1" H 5900 2800 60  0001 C CNN "MFP"
+F 6 "Panasonic ERA-6ARB752V" V 5900 2800 50  0001 C CNN "Alternative"
 	1    5900 2800
 	0    1    1    0
@@
 The LM399 has a\nTCR of 0.3 ppm/K
 Text Notes 5200 2500 0    60   ~ 0
-The output drift with the zener current\nis about 5 x 10^-3 ppm / ppm.\nIn order to meet the LM399 specs make sure the resistor\nhas a maximum TCR of 5 ppm / K (results in 0.03 ppm / K).
+The output drift with the zener current\nis about 5 x 10^-3 ppm / ppm.\nIn order to meet the LM399 specs make sure the resistor\nhas a maximum TCR of 10 ppm / K (results in 0.06 ppm / K).
 Text HLabel 5800 3100 1    60   UnSpc ~ 0
 V+
@@
 	1    0    0    -1
 $EndComp
-Text Notes 7100 3400 0    60   ~ 0
-e.g. PCF0805-13-7K5-B-T1 (5 ppm),\nTE Connectivity RU73X2A7K5LTDF (2 ppm),\nVishay S102 (2 ppm)\n\nPCF0805-13-3K-B-T1. (5 ppm),\nVishay S102 (2 ppm)
 Text Notes 7350 5050 0    60   ~ 0
 DON'T use AVX! They will melt at the spec'ed temperature
@@
 Text Label 6900 6100 3    60   ~ 0
 V_zener+
-Text Label 4200 2800 1    60   ~ 0
+Text Label 4200 3200 1    60   ~ 0
 V_zener+
 $Comp
@@
 	4600 2800 4600 2850
 Wire Wire Line
-	3800 2900 3800 2450
-Wire Wire Line
-	3800 3900 3800 3700
+	4000 3300 4000 2850
+Wire Wire Line
+	4000 3900 4000 3700
 Wire Wire Line
 	2500 2500 2500 2950
@@
 	6900 6000 6900 6100
 Wire Wire Line
-	4200 2800 4200 2900
+	4200 3200 4200 3300
 Wire Wire Line
 	5050 2800 5050 3400
@@
 	0    1    1    0
 $EndComp
+Text Notes 7000 2950 0    60   ~ 0
+e.g. ERA-6ARB752V (10 ppm)\nPCF0805-13-7K5-B-T1 (5 ppm),\nTE Connectivity RU73X2A7K5LTDF (2 ppm),\nVishay S102 (2 ppm)
+Text Notes 7350 5500 0    60   ~ 0
+17k: Pin 1 -> Pin 2\nPin 1 is correctly\nmarked on the package
 $EndSCHEMATC

Commit message: Removed via from bypass capacitor pad
Parts:
- U3: Alternative (none) -> TI OPA277U
Changed lines of the file:
@@
 EESchema Schematic File Version 4
 LIBS:reference_board-cache
-EELAYER 29 0
+EELAYER 30 0
 EELAYER END
 $Descr A4 11693 8268
@@
 F 4 "Analog Devices" H 5900 4050 50  0001 C CNN "MFN"
 F 5 "LT1001CS8" H 5900 4050 50  0001 C CNN "MFP"
+F 6 "TI OPA277U" H 5900 4050 50  0001 C CNN "Alternative"
 	1    5900 4050
 	1    0    0    -1

Commit message: Updated to v3.1.2 Added part number of the socket (optional)
Parts:
- U2: Alternative (none) -> Use a TE 8060-1G12 socket to mount diodes for burn-in
Other:
- note added: "Note: Use a TE 8060-1G12 socket\nto mount diodes for burn-in"
Changed lines of the file:
@@
 F 4 "Analog Devices" H 4100 3500 60  0001 C CNN "MFN"
 F 5 "LM399AH" H 4100 3500 60  0001 C CNN "MFP"
+F 6 "Use a TE 8060-1G12 socket to mount diodes for burn-in" H 4100 3500 50  0001 C CNN "Alternative"
 	1    4100 3500
 	1    0    0    -1
@@
 Text HLabel 4000 3900 3    60   UnSpc ~ 0
 V_heater-
-Text HLabel 2500 2500 1    60   UnSpc ~ 0
+Text HLabel 2350 2100 1    60   UnSpc ~ 0
 V_zener+_force
 $Comp
@@
 Text Notes 5200 1950 0    60   ~ 0
 This resistor will supply the zener current.\nIt does not need to be exactely 3k, but a\nzener current of 1 mA or slightly above is\nrecommended.\nThis resistor needs to be matched if the\namplification is changed. Currently\nI_Zener = (10 V - 6.95 V) / 3k
-Text Notes 2750 3250 0    60   ~ 0
+Text Notes 2600 2850 0    60   ~ 0
 The LM399 has a\nTCR of 0.3 ppm/K
 Text Notes 5200 2500 0    60   ~ 0
@@
 NoConn ~ 6000 4350
 NoConn ~ 5900 4350
-Text HLabel 2800 2500 1    60   Output ~ 0
+Text HLabel 2650 2100 1    60   Output ~ 0
 V_zener+_sense
 $Comp
 L Device:Net-Tie_2 NT1
 U 1 1 5976DF85
-P 2800 2650
-F 0 "NT1" V 2754 2738 50  0000 L CNN
-F 1 "NET-TIE" V 2845 2738 50  0000 L CNN
-F 2 "Custom_footprints:NET-TIE-0.15mm" H 2800 2550 50  0001 C CNN
-F 3 "" H 2800 2650 60  0000 C CNN
-	1    2800 2650
+P 2650 2250
+F 0 "NT1" V 2604 2338 50  0000 L CNN
+F 1 "NET-TIE" V 2695 2338 50  0000 L CNN
+F 2 "Custom_footprints:NET-TIE-0.15mm" H 2650 2150 50  0001 C CNN
+F 3 "" H 2650 2250 60  0000 C CNN
+	1    2650 2250
 	0    1    1    0
 $EndComp
@@
 	0    1    1    0
 $EndComp
-Text Label 2500 2950 3    60   ~ 0
+Text Label 2350 2550 3    60   ~ 0
 V_zener+
 Text Label 6900 6100 3    60   ~ 0
@@
 	4000 3900 4000 3700
 Wire Wire Line
-	2500 2500 2500 2950
+	2350 2100 2350 2550
 Wire Wire Line
 	6200 4050 6900 4050
@@
 	4200 3700 4200 3800
 Wire Wire Line
-	2500 2950 2800 2750
-Wire Wire Line
-	2800 2550 2800 2500
+	2350 2550 2650 2350
+Wire Wire Line
+	2650 2150 2650 2100
 Wire Wire Line
 	6900 6000 6900 6100
@@
 Text Notes 7350 5500 0    60   ~ 0
 17k: Pin 1 -> Pin 2\nPin 1 is correctly\nmarked on the package
+Text Notes 2150 3600 0    60   ~ 0
+Note: Use a TE 8060-1G12 socket\nto mount diodes for burn-in
 $EndSCHEMATC

Commit message: Changed op amp to LT1001 Added startup circuit Board shrink Changed temperature sensor to TI TMP236 Added mounting hole
Parts:
- added D1: BAQ333, Diode_SMD:D_MicroMELF, symbol Device:D
- added R3: 10k, Resistor_SMD:R_0603_1608Metric, symbol Device:R
- R2: value 200k -> 30k; MFP RR0816P-204-D -> RR0816P-303-D
Connections:
- wire segments 43 -> 46
Other:
- note added: "Startup circuit:\nDoes not cause zener shift\nwith different V_zener+"
- note added: "This resistor will supply the zener current.\nIt does not need to be exactely 7.5k, but a\nzener current of 1 mA or slightly above is\nrecommended.\nThis resistor needs to be matched if the\namplification is changed. Currently\nI_Zener = (15 V - 6.95 V) / 7.5k"
- note removed: "This resistor will supply the zener current.\nIt does not need to be exactely 3k, but a\nzener current of 1 mA or slightly above is\nrecommended.\nThis resistor needs to be matched if the\namplification is changed. Currently\nI_Zener = (10 V - 6.95 V) / 3k"
- moved on the sheet: U2
Changed lines of the file:
@@
 Sheet 2 2
 Title "LM399 negative voltage reference"
-Date "2019-06-28"
-Rev "v3.1.1"
+Date "2019-11-20"
+Rev "v3.2.0"
 Comp ""
 Comment1 "Copyright (©) 2018, Patrick Baus <patrick.baus@physik.tu-darmstadt.de>"
@@
 L Reference_Voltage:LM399 U2
 U 1 1 591A5398
-P 4100 3500
+P 3500 3500
 AR Path="/591A5398" Ref="U2"  Part="1"
 AR Path="/591A50E3/591A5398" Ref="U2"  Part="1"
-F 0 "U2" H 4300 3550 60  0000 L CNN
-F 1 "LM399" H 4300 3450 60  0000 L CNN
-F 2 "Custom_footprints:TO-46-4_ThermalShield" H 4100 3450 60  0001 C CNN
-F 3 "" H 4100 3450 60  0001 C CNN
-F 4 "Analog Devices" H 4100 3500 60  0001 C CNN "MFN"
-F 5 "LM399AH" H 4100 3500 60  0001 C CNN "MFP"
-F 6 "Use a TE 8060-1G12 socket to mount diodes for burn-in" H 4100 3500 50  0001 C CNN "Alternative"
-	1    4100 3500
-	1    0    0    -1
-$EndComp
-Text HLabel 4000 2850 1    60   UnSpc ~ 0
+F 0 "U2" H 3700 3550 60  0000 L CNN
+F 1 "LM399" H 3700 3450 60  0000 L CNN
+F 2 "Custom_footprints:TO-46-4_ThermalShield" H 3500 3450 60  0001 C CNN
+F 3 "" H 3500 3450 60  0001 C CNN
+F 4 "Analog Devices" H 3500 3500 60  0001 C CNN "MFN"
+F 5 "LM399AH" H 3500 3500 60  0001 C CNN "MFP"
+F 6 "Use a TE 8060-1G12 socket to mount diodes for burn-in" H 3500 3500 50  0001 C CNN "Alternative"
+	1    3500 3500
+	1    0    0    -1
+$EndComp
+Text HLabel 3400 2850 1    60   UnSpc ~ 0
 V-heater+
-Text HLabel 4000 3900 3    60   UnSpc ~ 0
+Text HLabel 3400 3900 3    60   UnSpc ~ 0
 V_heater-
-Text HLabel 2350 2100 1    60   UnSpc ~ 0
+Text HLabel 1750 2250 1    60   UnSpc ~ 0
 V_zener+_force
 $Comp
@@
 $EndComp
 Text Notes 5200 1950 0    60   ~ 0
-This resistor will supply the zener current.\nIt does not need to be exactely 3k, but a\nzener current of 1 mA or slightly above is\nrecommended.\nThis resistor needs to be matched if the\namplification is changed. Currently\nI_Zener = (10 V - 6.95 V) / 3k
-Text Notes 2600 2850 0    60   ~ 0
+This resistor will supply the zener current.\nIt does not need to be exactely 7.5k, but a\nzener current of 1 mA or slightly above is\nrecommended.\nThis resistor needs to be matched if the\namplification is changed. Currently\nI_Zener = (15 V - 6.95 V) / 7.5k
+Text Notes 2000 3000 0    60   ~ 0
 The LM399 has a\nTCR of 0.3 ppm/K
 Text Notes 5200 2500 0    60   ~ 0
@@
 	1    0    0    -1
 $EndComp
-Text Notes 1850 4000 0    60   ~ 0
+Text Notes 1250 4000 0    60   ~ 0
 TODO:\n- use 4 drill holes to mount styrofoam
 Text Notes 7350 4900 0    60   ~ 0
@@
 Text Notes 4300 6300 0    60   ~ 0
 Kelvin connect this to the V_zener+ input pin
-Text Notes 3150 1200 0    60   ~ 0
+Text Notes 1400 900  0    60   ~ 0
 Use 1 oz./sqft of copper to\nminimize trace resistance and\ntherefore minimize succeptibility\nto temperature.
-Text Notes 3200 1650 0    60   ~ 0
+Text Notes 1400 1300 0    60   ~ 0
 Trace resistance of 0.32 Ohm\n(100mm, 4000 ppm / K) causes\na 1.5 µV / K error.
 NoConn ~ 6000 4350
 NoConn ~ 5900 4350
-Text HLabel 2650 2100 1    60   Output ~ 0
+Text HLabel 2050 2250 1    60   Output ~ 0
 V_zener+_sense
 $Comp
 L Device:Net-Tie_2 NT1
 U 1 1 5976DF85
-P 2650 2250
-F 0 "NT1" V 2604 2338 50  0000 L CNN
-F 1 "NET-TIE" V 2695 2338 50  0000 L CNN
-F 2 "Custom_footprints:NET-TIE-0.15mm" H 2650 2150 50  0001 C CNN
-F 3 "" H 2650 2250 60  0000 C CNN
-	1    2650 2250
+P 2050 2400
+F 0 "NT1" V 2004 2488 50  0000 L CNN
+F 1 "NET-TIE" V 2095 2488 50  0000 L CNN
+F 2 "Custom_footprints:NET-TIE-0.15mm" H 2050 2300 50  0001 C CNN
+F 3 "" H 2050 2400 60  0000 C CNN
+	1    2050 2400
 	0    1    1    0
 $EndComp
@@
 	0    1    1    0
 $EndComp
-Text Label 2350 2550 3    60   ~ 0
+Text Label 1750 2700 3    60   ~ 0
 V_zener+
 Text Label 6900 6100 3    60   ~ 0
 V_zener+
-Text Label 4200 3200 1    60   ~ 0
+Text Label 3600 3200 1    60   ~ 0
 V_zener+
 $Comp
@@
 	0    1    1    0
 $EndComp
-Text Notes 950  4800 0    60   ~ 0
+Text Notes 700  4800 0    60   ~ 0
 Kelvin connect the Zener. Even the the small current\npassing through R1 (1 mA) will introduce an error of 0.2 ppm/K\ngiven a normal PCB copper trace.\n(10 mm trace 0=> 0.2 ohm, 1 mA, 0.7 % tcr, ~~7 V reference)
 Text Notes 1950 5600 0    60   ~ 0
@@
 Text Notes 8350 3800 0    60   ~ 0
 Information on insulation resistance can be found here:\nhttp://www.iequalscdvdt.com/Insulation_resis_.html\nhttps://www.vishay.com/docs/26033/gentechinfofilm.pdf
-$Comp
-L Device:R R2
-U 1 1 59E8CFD2
-P 4850 2800
-F 0 "R2" V 4643 2800 50  0000 C CNN
-F 1 "200k" V 4734 2800 50  0000 C CNN
-F 2 "Resistor_SMD:R_0603_1608Metric" V 4780 2800 50  0001 C CNN
-F 3 "" H 4850 2800 50  0001 C CNN
-F 4 "Susumu" H 4850 2800 60  0001 C CNN "MFN"
-F 5 "RR0816P-204-D" H 4850 2800 60  0001 C CNN "MFP"
-	1    4850 2800
-	0    1    1    0
-$EndComp
-Text HLabel 4600 2850 3    60   UnSpc ~ 0
-V-
-Connection ~ 5050 2800
-Wire Wire Line
-	4600 2800 4600 2850
-Wire Wire Line
-	4000 3300 4000 2850
-Wire Wire Line
-	4000 3900 4000 3700
-Wire Wire Line
-	2350 2100 2350 2550
+Wire Wire Line
+	3400 3300 3400 2850
+Wire Wire Line
+	3400 3900 3400 3700
+Wire Wire Line
+	1750 2250 1750 2700
 Wire Wire Line
 	6200 4050 6900 4050
@@
 	5450 4150 5600 4150
 Wire Wire Line
-	4200 3950 5600 3950
-Wire Wire Line
-	5000 2800 5050 2800
+	3600 3950 5600 3950
 Wire Wire Line
 	6050 2800 6900 2800
@@
 Connection ~ 5800 4500
 Wire Wire Line
-	4200 3700 4200 3800
-Wire Wire Line
-	2350 2550 2650 2350
-Wire Wire Line
-	2650 2150 2650 2100
+	3600 3700 3600 3800
+Wire Wire Line
+	1750 2700 2050 2500
+Wire Wire Line
+	2050 2300 2050 2250
 Wire Wire Line
 	6900 6000 6900 6100
 Wire Wire Line
-	4200 3200 4200 3300
+	3600 3200 3600 3300
 Wire Wire Line
 	5050 2800 5050 3400
@@
 	5050 3600 5050 3800
 Wire Wire Line
-	5050 3800 4200 3800
-Connection ~ 4200 3800
+	5050 3800 3600 3800
+Connection ~ 3600 3800
 Wire Wire Line
 	6900 4800 6550 4800
@@
 	6550 5350 6550 5200
 Connection ~ 6550 5350
-Wire Wire Line
-	4700 2800 4600 2800
 Text Notes 8400 1950 0    60   ~ 0
 Mount the LM399 a *little* off the board,\nto keep stress away.\nSource: http://www.eevblog.com/forum/\nmetrology/ultra-precision-reference-ltz1000/\nmsg404500/#msg404500
@@
 	5800 4500 5800 5050
 Wire Wire Line
-	4200 3800 4200 3950
+	3600 3800 3600 3950
 Wire Wire Line
 	6550 5350 6750 5350
@@
 Text Notes 7350 5500 0    60   ~ 0
 17k: Pin 1 -> Pin 2\nPin 1 is correctly\nmarked on the package
-Text Notes 2150 3600 0    60   ~ 0
+Text Notes 1550 3600 0    60   ~ 0
 Note: Use a TE 8060-1G12 socket\nto mount diodes for burn-in
+$Comp
+L power:GND #PWR0103
+U 1 1 5DD6028A
+P 4300 3200
+F 0 "#PWR0103" H 4300 2950 50  0001 C CNN
+F 1 "GND" H 4305 3027 50  0000 C CNN
+F 2 "" H 4300 3200 50  0001 C CNN
+F 3 "" H 4300 3200 50  0001 C CNN
+	1    4300 3200
+	1    0    0    -1
+$EndComp
+Wire Wire Line
+	4300 3200 4300 3150
+$Comp
+L Device:R R3
+U 1 1 5DD610DD
+P 4300 2600
+F 0 "R3" H 4400 2650 50  0000 L CNN
+F 1 "10k" H 4400 2550 50  0000 L CNN
+F 2 "Resistor_SMD:R_0603_1608Metric" V 4230 2600 50  0001 C CNN
+F 3 "~" H 4300 2600 50  0001 C CNN
+F 4 "Susumu" H 4300 2600 50  0001 C CNN "MFN"
+F 5 "RR0816P-103-D" H 4300 2600 50  0001 C CNN "MFP"
+	1    4300 2600
+	1    0    0    -1
+$EndComp
+$Comp
+L Device:R R2
+U 1 1 5DD614F5
+P 4300 3000
+F 0 "R2" H 4400 3050 50  0000 L CNN
+F 1 "30k" H 4400 2950 50  0000 L CNN
+F 2 "Resistor_SMD:R_0603_1608Metric" V 4230 3000 50  0001 C CNN
+F 3 "~" H 4300 3000 50  0001 C CNN
+F 4 "Susumu" H 4300 3000 50  0001 C CNN "MFN"
+F 5 "RR0816P-303-D" H 4300 3000 50  0001 C CNN "MFP"
+	1    4300 3000
+	1    0    0    -1
+$EndComp
+Text HLabel 4300 2350 1    60   UnSpc ~ 0
+V_zener+_force
+Wire Wire Line
+	4300 2350 4300 2450
+Wire Wire Line
+	4300 2750 4300 2800
+$Comp
+L Device:D D1
+U 1 1 5DD64006
+P 4850 2800
+F 0 "D1" H 4850 3050 50  0000 C CNN
+F 1 "BAQ333" H 4850 2950 50  0000 C CNN
+F 2 "Diode_SMD:D_MicroMELF" H 4850 2800 50  0001 C CNN
+F 3 "~" H 4850 2800 50  0001 C CNN
+F 4 "Vishay" H 4850 2800 50  0001 C CNN "MFN"
+F 5 "BAQ333-TR" H 4850 2800 50  0001 C CNN "MFP"
+	1    4850 2800
+	1    0    0    -1
+$EndComp
+Wire Wire Line
+	5050 2800 5000 2800
+Connection ~ 5050 2800
+Wire Wire Line
+	4700 2800 4300 2800
+Connection ~ 4300 2800
+Wire Wire Line
+	4300 2800 4300 2850
+Wire Notes Line
+	4000 1500 4950 1500
+Wire Notes Line
+	4950 1500 4950 3500
+Wire Notes Line
+	4950 3500 4000 3500
+Wire Notes Line
+	4000 3500 4000 1500
+Text Notes 3800 1400 0    60   ~ 0
+Startup circuit:\nDoes not cause zener shift\nwith different V_zener+
 $EndSCHEMATC
