File: LM399.sch (KiCad schematic (older format))
At the start: 15 parts, among them U2 LM399, U3 LT1001

Commit message: Updated to v.3.2.1 -Changed D1 to a plastic package to eliminate possible light sensitivity -Updated bom.ini for the latest version of KiBOM -Updated symbol fields (changed MFP -> PN) for KiCost compatibility -Added PCBA config -Updated Gerber files
Parts:
- C1, C2, C3: MFP GRM31C5C1H104JA01L -> (none); PN (none) -> GRM31C5C1H104JA01L
- D1: value BAQ333 -> BAS116; footprint Diode_SMD:D_MicroMELF -> Diode_SMD:D_SOD-123; MFN Vishay -> Nexperia; MFP BAQ333-TR -> (none); Note (none) -> Use a plastic package to eliminate light sensitivity; PN (none) -> BAS116GWJ
- R1: MFP PCF0805-13-7K5-B-T1 -> (none); PN (none) -> PCF0805-13-7K5-B-T1
- R2: MFP RR0816P-303-D -> (none); PN (none) -> RR0816P-303-D
- R3: MFP RR0816P-103-D -> (none); PN (none) -> RR0816P-103-D
- RN1: Config (none) -> -PCBA; MFP 300144Z -> (none); Note (none) -> Vishay 300144Z, 0.1% abs. tol. 0.1% ratio tol.; PN (none) -> Y1691V0689BB9L
- U2: Alternative Use a TE 8060-1G12 socket to mount diodes for burn-in -> (none); Config (none) -> -PCBA; MFP LM399AH -> (none); Note (none) -> Use a TE 8060-1G12 socket to mount diodes for burn-in; PN (none) -> LM399AH
- U3: MFP LT1001CS8 -> (none); PN (none) -> LT1001CS8
Other:
- note added: "Voltage here should be a few Volts above (Vreg-7V)"
- note removed: "17k: Pin 1 -> Pin 2\nPin 1 is correctly\nmarked on the package"
- note removed: "DON'T use AVX! They will melt at the spec'ed temperature"
- note removed: "Information on insulation resistance can be found here:\nhttp://www.iequalscdvdt.com/Insulation_resis_.html\nhttps://www.vishay.com/docs/26033/gentechinfofilm.pdf"
- note removed: "Kelvin connect the Zener. Even the the small current\npassing through R1 (1 mA) will introduce an error of 0.2 ppm/K\ngiven a normal PCB copper trace.\n(10 mm trace 0=> 0.2 ohm, 1 mA, 0.7 % tcr, ~~7 V reference)"
- note removed: "Kelvin connect this to the V_zener+ input pin"
- note removed: "Mount the LM399 a *little* off the board,\nto keep stress away.\nSource: http://www.eevblog.com/forum/\nmetrology/ultra-precision-reference-ltz1000/\nmsg404500/#msg404500"
- note removed: "Note: Use a TE 8060-1G12 socket\nto mount diodes for burn-in"
- note removed: "Output voltage Table:\nVoltage | R1 | R2 | R3\n------------------\n-10 V | 3k | 9k | 20k\n-15 V | 7.89k | 20k | 17k"
- note removed: "TODO:\n- use 4 drill holes to mount styrofoam"
- note removed: "The LM399 has a\nTCR of 0.3 ppm/K"
- note removed: "The output drift with the zener current\nis about 5 x 10^-3 ppm / ppm.\nIn order to meet the LM399 specs make sure the resistor\nhas a maximum TCR of 10 ppm / K (results in 0.06 ppm / K)."
- note removed: "This resistor will supply the zener current.\nIt does not need to be exactely 7.5k, but a\nzener current of 1 mA or slightly above is\nrecommended.\nThis resistor needs to be matched if the\namplification is changed. Currently\nI_Zener = (15 V - 6.95 V) / 7.5k"
- note removed: "Trace resistance of 0.32 Ohm\n(100mm, 4000 ppm / K) causes\na 1.5 µV / K error."
- note removed: "Use 1 oz./sqft of copper to\nminimize trace resistance and\ntherefore minimize succeptibility\nto temperature."
- note removed: "Use a Film capacitor with a high insulation\nresistance (no polyester), which is stable\nover temperature. Nowadays C0G (BME) is\neven better than film."
- note removed: "e.g. ERA-6ARB752V (10 ppm)\nPCF0805-13-7K5-B-T1 (5 ppm),\nTE Connectivity RU73X2A7K5LTDF (2 ppm),\nVishay S102 (2 ppm)"
- moved on the sheet: C1, C2, C3, R1, R2, R3, RN1, U2, U3

Commit message: Updated footprints and 3d models in preparation for KiCAD 5.1.7 (which contains an LM399 footprint, see https://github.com/KiCad/kicad-footprints/pull/2481)
Parts:
- U2: footprint Custom_footprints:TO-46-4_ThermalShield -> Custom_footprints:Analog_TO-46-4_ThermalShield; Note Use a TE 8060-1G12 socket to mount diodes for burn-in -> Use a TE 8060-1G12 or TE 8060-G22 socket to mount diodes fo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
Other:
- note added: "17k: Pin 1 <-> Pin 2\n20k: Pin 2 <-> Pin 3\nPin 1 is marked on\nthe package"
- note added: "Kelvin connect the Zener. Even the the small current\npassing through R1 (1 mA) will introduce an error of 0.2 ppm/K\ngiven a normal PCB copper trace.\n(10 mm trace 0=> 0.2 ohm, 1 mA, 0.7 % tcr, ~~7 V reference)"
- note added: "Kelvin connect this to the V_zener+ input pin"
- note added: "Mount the LM399 a *little* off the board,\nto keep stress away.\nSource: http://www.eevblog.com/forum/\nmetrology/ultra-precision-reference-ltz1000/\nmsg404500/#msg404500"
- note added: "Note: Use a TE 8060-1G12\nor 8060-1G22 socket to\nmount diodes for burn-in.\nThe 1G22 is smaller in\nheight, but harder to get."
- note added: "Output voltage Table:\nVoltage | R1 | R2 | R3\n------------------\n-10 V | 3k | 9k | 20k\n-15 V | 7.5k | 20k | 17k"
- note added: "The LM399 has a\nTCR of 0.3 ppm/K"
- note added: "The output drift with the zener current\nis about 0.15 ppm / ppm maximum.\nIn order to meet the LM399 specs make sure the resistor\nhas a maximum TCR of 10 ppm / K (results in 1.5 ppm / K)."
- note added: "This resistor will supply the zener current.\nIt does not need to be exactely 7.5k, but a\nzener current of 1 mA or slightly above is\nrecommended.\nThis resistor needs to be matched if the\namplification is changed. Currently\nI_Zener = (15 V - 6.95 V) / 7.5k"
- note added: "Trace resistance of 0.32 Ohm\n(100mm, 4000 ppm / K) causes\na 1.5 µV / K error."
- note added: "Use 1 oz./sqft of copper to\nminimize trace resistance and\ntherefore minimize succeptibility\nto temperature."
- note added: "Use a Film capacitor with a high insulation\nresistance (no polyester), which is stable\nover temperature. Nowadays C0G (BME) is\neven better than film.\nInformation on insulation resistance can be found here:\nhttp://www.iequalscdvdt.com/Insulation_resis_.html\nhttps://www.vishay.com/docs/26033/gentechinfofilm.pdf"
- note added: "e.g. ERA-6ARB752V (10 ppm)\nPCF0805-13-7K5-B-T1 (5 ppm),\nTE Connectivity RU73X2A7K5LTDF (2 ppm),\nVishay S102 (2 ppm)"
Changed lines of the file:
@@
 Title "LM399 negative voltage reference"
 Date "2019-11-20"
-Rev "v3.2.0"
+Rev "v3.2.2"
 Comp ""
 Comment1 "Copyright (©) 2020, Patrick Baus <patrick.baus@physik.tu-darmstadt.de>"
@@
 F 0 "U2" H 3750 3100 60  0000 L CNN
 F 1 "LM399" H 3750 3000 60  0000 L CNN
-F 2 "Custom_footprints:TO-46-4_ThermalShield" H 3550 3000 60  0001 C CNN
+F 2 "Custom_footprints:Analog_TO-46-4_ThermalShield" H 3550 3000 60  0001 C CNN
 F 3 "https://www.analog.com/media/en/technical-documentation/data-sheets/199399fc.pdf" H 3550 3000 60  0001 C CNN
 F 4 "Analog Devices" H 3550 3050 60  0001 C CNN "MFN"
 F 5 "LM399AH" H 3550 3050 50  0001 C CNN "PN"
-F 6 "Use a TE 8060-1G12 socket to mount diodes for burn-in" H 3550 3050 50  0001 C CNN "Note"
+F 6 "Use a TE 8060-1G12 or TE 8060-G22 socket to mount diodes for burn-in" H 3550 3050 50  0001 C CNN "Note"
 F 7 "-PCBA" H 3550 3050 50  0001 C CNN "Config"
 	1    3550 3050
@@
 Text Notes 5250 1950 0    60   ~ 0
 Voltage here should be a few Volts above (Vreg-7V)
+Text Notes 2350 950  0    60   ~ 0
+Use 1 oz./sqft of copper to\nminimize trace resistance and\ntherefore minimize succeptibility\nto temperature.
+Text Notes 2350 1350 0    60   ~ 0
+Trace resistance of 0.32 Ohm\n(100mm, 4000 ppm / K) causes\na 1.5 µV / K error.
+Text Notes 2350 2850 0    60   ~ 0
+The LM399 has a\nTCR of 0.3 ppm/K
+Text Notes 1950 3430 0    60   ~ 0
+Note: Use a TE 8060-1G12\nor 8060-1G22 socket to\nmount diodes for burn-in.\nThe 1G22 is smaller in\nheight, but harder to get.
+Text Notes 1150 5200 0    60   ~ 0
+Kelvin connect the Zener. Even the the small current\npassing through R1 (1 mA) will introduce an error of 0.2 ppm/K\ngiven a normal PCB copper trace.\n(10 mm trace 0=> 0.2 ohm, 1 mA, 0.7 % tcr, ~~7 V reference)
+Text Notes 2050 6000 0    60   ~ 0
+Output voltage Table:\nVoltage   | R1    | R2  | R3\n------------------\n-10 V    | 3k    | 9k  | 20k\n-15 V    | 7.5k  | 20k | 17k
+Text Notes 7850 2700 0    60   ~ 0
+This resistor will supply the zener current.\nIt does not need to be exactely 7.5k, but a\nzener current of 1 mA or slightly above is\nrecommended.\nThis resistor needs to be matched if the\namplification is changed. Currently\nI_Zener = (15 V - 6.95 V) / 7.5k
+Wire Notes Line
+	6250 2250 7750 2250
+Wire Notes Line
+	6250 2250 6300 2300
+Wire Notes Line
+	6250 2250 6300 2200
+Text Notes 7850 3200 0    60   ~ 0
+The output drift with the zener current\nis about 0.15 ppm / ppm maximum.\nIn order to meet the LM399 specs make sure the resistor\nhas a maximum TCR of 10 ppm / K (results in 1.5 ppm / K).
+Text Notes 8450 3600 0    60   ~ 0
+e.g. ERA-6ARB752V (10 ppm)\nPCF0805-13-7K5-B-T1 (5 ppm),\nTE Connectivity RU73X2A7K5LTDF (2 ppm),\nVishay S102 (2 ppm)
+Text Notes 7650 4650 0    60   ~ 0
+Use a Film capacitor with a high insulation\nresistance (no polyester), which is stable\nover temperature. Nowadays C0G (BME) is\neven better than film.\nInformation on insulation resistance can be found here:\nhttp://www.iequalscdvdt.com/Insulation_resis_.html\nhttps://www.vishay.com/docs/26033/gentechinfofilm.pdf
+Text Notes 7650 5150 0    60   ~ 0
+17k: Pin 1 <-> Pin 2\n20k: Pin 2 <-> Pin 3\nPin 1 is marked on\nthe package
+Text Notes 4750 5500 0    60   ~ 0
+Kelvin connect this to the V_zener+ input pin
+Text Notes 7850 1550 0    60   ~ 0
+Mount the LM399 a *little* off the board,\nto keep stress away.\nSource: http://www.eevblog.com/forum/\nmetrology/ultra-precision-reference-ltz1000/\nmsg404500/#msg404500
 $EndSCHEMATC

Commit message: Added ibom Simplified RN1 description Moved R2 a little bit away from R3 to prevent problems during soldering
Other:
- note added: "Output voltage Table:\nVoltage | R1 | RN1a | RN1b\n-----------------------\n-10 V | 3k | 20k | 9k\n-15 V | 7.5k | 17k | 20k"
- note removed: "Output voltage Table:\nVoltage | R1 | R2 | R3\n------------------\n-10 V | 3k | 9k | 20k\n-15 V | 7.5k | 20k | 17k"
Changed lines of the file:
@@
 Kelvin connect the Zener. Even the the small current\npassing through R1 (1 mA) will introduce an error of 0.2 ppm/K\ngiven a normal PCB copper trace.\n(10 mm trace 0=> 0.2 ohm, 1 mA, 0.7 % tcr, ~~7 V reference)
 Text Notes 2050 6000 0    60   ~ 0
-Output voltage Table:\nVoltage   | R1    | R2  | R3\n------------------\n-10 V    | 3k    | 9k  | 20k\n-15 V    | 7.5k  | 20k | 17k
+Output voltage Table:\nVoltage   | R1    | RN1a  | RN1b\n-----------------------\n-10 V    | 3k    |   20k  | 9k\n-15 V    | 7.5k  |   17k  | 20k
 Text Notes 7850 2700 0    60   ~ 0
 This resistor will supply the zener current.\nIt does not need to be exactely 7.5k, but a\nzener current of 1 mA or slightly above is\nrecommended.\nThis resistor needs to be matched if the\namplification is changed. Currently\nI_Zener = (15 V - 6.95 V) / 7.5k

Commit message: Replaced startup circuit with a JFET
Parts:
- removed D1: BAS116, Diode_SMD:D_SOD-123, symbol Device:D
- removed R2: 30k, Resistor_SMD:R_0603_1608Metric, symbol Device:R
- removed R3: 10k, Resistor_SMD:R_0603_1608Metric, symbol Device:R
- added Q?: J270, Package_TO_SOT_SMD:SOT-23, symbol Device:Q_PJFET_DSG
- added R?: 2k, Resistor_SMD:R_0603_1608Metric, symbol Device:R
Connections:
- wire segments 46 -> 45
Other:
- note added: "Startup circuit:\nIt does not cause zener shift\nwith different V_zener+\nThe gate of the JFET is held\nat the positive supply of the zener.\nThe JFET will therefore conduct and\npull the negative leg of the zener down\nuntil the its source (the negative leg of\nthe zener) is abour 2 V to 4 V below the\nsupply. It will then turn off and leakage\nwill be on the order of a few pA.\nThe 2k resistor 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"
- note removed: "Startup circuit:\nDoes not cause zener shift\nwith different V_zener+"
- note removed: "Voltage here should be a few Volts above (Vreg-7V)"
- moved on the sheet: U2
Changed lines of the file:
@@
 Sheet 2 2
 Title "LM399 negative voltage reference"
-Date "2019-11-20"
-Rev "v3.2.2"
+Date "2021-05-20"
+Rev "v3.3.0"
 Comp ""
 Comment1 "Copyright (©) 2020, Patrick Baus <patrick.baus@physik.tu-darmstadt.de>"
@@
 L Reference_Voltage:LM399 U2
 U 1 1 591A5398
-P 3550 3050
+P 3000 3050
 AR Path="/591A5398" Ref="U2"  Part="1"
 AR Path="/591A50E3/591A5398" Ref="U2"  Part="1"
-F 0 "U2" H 3750 3100 60  0000 L CNN
-F 1 "LM399" H 3750 3000 60  0000 L CNN
-F 2 "Custom_footprints:Analog_TO-46-4_ThermalShield" H 3550 3000 60  0001 C CNN
-F 3 "https://www.analog.com/media/en/technical-documentation/data-sheets/199399fc.pdf" H 3550 3000 60  0001 C CNN
-F 4 "Analog Devices" H 3550 3050 60  0001 C CNN "MFN"
-F 5 "LM399AH" H 3550 3050 50  0001 C CNN "PN"
-F 6 "Use a TE 8060-1G12 or TE 8060-G22 socket to mount diodes for burn-in" H 3550 3050 50  0001 C CNN "Note"
-F 7 "-PCBA" H 3550 3050 50  0001 C CNN "Config"
-	1    3550 3050
-	1    0    0    -1
-$EndComp
-Text HLabel 3450 2400 1    60   UnSpc ~ 0
+F 0 "U2" H 3200 3100 60  0000 L CNN
+F 1 "LM399" H 3200 3000 60  0000 L CNN
+F 2 "Custom_footprints:Analog_TO-46-4_ThermalShield" H 3000 3000 60  0001 C CNN
+F 3 "https://www.analog.com/media/en/technical-documentation/data-sheets/199399fc.pdf" H 3000 3000 60  0001 C CNN
+F 4 "Analog Devices" H 3000 3050 60  0001 C CNN "MFN"
+F 5 "LM399AH" H 3000 3050 50  0001 C CNN "PN"
+F 6 "Use a TE 8060-1G12 or TE 8060-G22 socket to mount diodes for burn-in" H 3000 3050 50  0001 C CNN "Note"
+F 7 "-PCBA" H 3000 3050 50  0001 C CNN "Config"
+	1    3000 3050
+	1    0    0    -1
+$EndComp
+Text HLabel 2900 2400 1    60   UnSpc ~ 0
 V-heater+
-Text HLabel 3450 3450 3    60   UnSpc ~ 0
+Text HLabel 2900 3450 3    60   UnSpc ~ 0
 V_heater-
 Text HLabel 4300 4550 1    60   UnSpc ~ 0
@@
 Text Label 6950 5650 3    60   ~ 0
 V_zener+
-Text Label 3650 2750 1    60   ~ 0
+Text Label 3100 2750 1    60   ~ 0
 V_zener+
 $Comp
@@
 $EndComp
 Wire Wire Line
-	3450 2850 3450 2400
-Wire Wire Line
-	3450 3450 3450 3250
+	2900 2850 2900 2400
+Wire Wire Line
+	2900 3450 2900 3250
 Wire Wire Line
 	4300 4550 4300 5000
@@
 	5500 3700 5650 3700
 Wire Wire Line
-	3650 3500 5650 3500
+	3100 3500 5650 3500
 Wire Wire Line
 	6100 2350 6950 2350
@@
 Connection ~ 5850 4050
 Wire Wire Line
-	3650 3250 3650 3350
+	3100 3250 3100 3350
 Wire Wire Line
 	4300 5000 4600 4800
@@
 	6950 5550 6950 5650
 Wire Wire Line
-	3650 2750 3650 2850
+	3100 2750 3100 2850
 Wire Wire Line
 	5100 2350 5100 2950
@@
 	5100 3150 5100 3350
 Wire Wire Line
-	5100 3350 3650 3350
-Connection ~ 3650 3350
+	5100 3350 3100 3350
+Connection ~ 3100 3350
 Wire Wire Line
 	6950 4350 6600 4350
@@
 	5850 4050 5850 4600
 Wire Wire Line
-	3650 3350 3650 3500
+	3100 3350 3100 3500
 Wire Wire Line
 	6600 4900 6800 4900
@@
 	0    1    1    0
 $EndComp
-$Comp
-L power:GND #PWR0103
-U 1 1 5DD6028A
-P 4350 2750
-F 0 "#PWR0103" H 4350 2500 50  0001 C CNN
-F 1 "GND" H 4355 2577 50  0000 C CNN
-F 2 "" H 4350 2750 50  0001 C CNN
-F 3 "" H 4350 2750 50  0001 C CNN
-	1    4350 2750
-	1    0    0    -1
-$EndComp
-Wire Wire Line
-	4350 2750 4350 2700
-$Comp
-L Device:R R3
-U 1 1 5DD610DD
-P 4350 2150
-F 0 "R3" H 4450 2200 50  0000 L CNN
-F 1 "10k" H 4450 2100 50  0000 L CNN
-F 2 "Resistor_SMD:R_0603_1608Metric" V 4280 2150 50  0001 C CNN
-F 3 "~" H 4350 2150 50  0001 C CNN
-F 4 "Susumu" H 4350 2150 50  0001 C CNN "MFN"
-F 5 "RR0816P-103-D" H 4350 2150 50  0001 C CNN "PN"
-	1    4350 2150
-	1    0    0    -1
-$EndComp
-$Comp
-L Device:R R2
-U 1 1 5DD614F5
-P 4350 2550
-F 0 "R2" H 4450 2600 50  0000 L CNN
-F 1 "30k" H 4450 2500 50  0000 L CNN
-F 2 "Resistor_SMD:R_0603_1608Metric" V 4280 2550 50  0001 C CNN
-F 3 "~" H 4350 2550 50  0001 C CNN
-F 4 "Susumu" H 4350 2550 50  0001 C CNN "MFN"
-F 5 "RR0816P-303-D" H 4350 2550 50  0001 C CNN "PN"
-	1    4350 2550
-	1    0    0    -1
-$EndComp
-Text HLabel 4350 1900 1    60   UnSpc ~ 0
+Text HLabel 4450 2800 0    60   UnSpc ~ 0
 V_zener+_force
-Wire Wire Line
-	4350 1900 4350 2000
-Wire Wire Line
-	4350 2300 4350 2350
-$Comp
-L Device:D D1
-U 1 1 5DD64006
-P 4900 2350
-F 0 "D1" H 4900 2600 50  0000 C CNN
-F 1 "BAS116" H 4900 2500 50  0000 C CNN
-F 2 "Diode_SMD:D_SOD-123" H 4900 2350 50  0001 C CNN
-F 3 "https://assets.nexperia.com/documents/data-sheet/BAS116GW.pdf" H 4900 2350 50  0001 C CNN
-F 4 "Nexperia" H 4900 2350 50  0001 C CNN "MFN"
-F 5 "Use a plastic package to eliminate light sensitivity" H 4900 2350 50  0001 C CNN "Note"
-F 6 "BAS116GWJ" H 4900 2350 50  0001 C CNN "PN"
-	1    4900 2350
-	1    0    0    -1
-$EndComp
-Wire Wire Line
-	5100 2350 5050 2350
 Connection ~ 5100 2350
-Wire Wire Line
-	4750 2350 4350 2350
-Connection ~ 4350 2350
-Wire Wire Line
-	4350 2350 4350 2400
-Wire Notes Line
-	4050 1050 5000 1050
-Wire Notes Line
-	5000 1050 5000 3050
-Wire Notes Line
-	5000 3050 4050 3050
-Wire Notes Line
-	4050 3050 4050 1050
-Text Notes 5100 1700 0    60   ~ 0
-Startup circuit:\nDoes not cause zener shift\nwith different V_zener+
-Wire Notes Line
-	4650 2300 4650 1900
-Wire Notes Line
-	4650 1900 5200 1900
-Wire Notes Line
-	4650 2300 4700 2250
-Wire Notes Line
-	4650 2300 4600 2250
-Text Notes 5250 1950 0    60   ~ 0
-Voltage here should be a few Volts above (Vreg-7V)
+Wire Notes Line
+	3600 2000 5000 2000
+Wire Notes Line
+	5000 2000 5000 3050
+Wire Notes Line
+	5000 3050 3600 3050
+Wire Notes Line
+	3600 3050 3600 2000
+Text Notes 4100 1850 0    60   ~ 0
+Startup circuit:\nIt does not cause zener shift\nwith different V_zener+\nThe gate of the JFET is held\nat the positive supply of the zener.\nThe JFET will therefore conduct and\npull the negative leg of the zener down\nuntil the its source (the negative leg of\nthe zener) is abour 2 V to 4 V below the\nsupply. It will then turn off and leakage\nwill be on the order of a few pA.\nThe 2k resistor is for protection only.
 Text Notes 2350 950  0    60   ~ 0
 Use 1 oz./sqft of copper to\nminimize trace resistance and\ntherefore minimize succeptibility\nto temperature.
 Text Notes 2350 1350 0    60   ~ 0
 Trace resistance of 0.32 Ohm\n(100mm, 4000 ppm / K) causes\na 1.5 µV / K error.
-Text Notes 2350 2850 0    60   ~ 0
+Text Notes 1800 2850 0    60   ~ 0
 The LM399 has a\nTCR of 0.3 ppm/K
-Text Notes 1950 3430 0    60   ~ 0
+Text Notes 1400 3430 0    60   ~ 0
 Note: Use a TE 8060-1G12\nor 8060-1G22 socket to\nmount diodes for burn-in.\nThe 1G22 is smaller in\nheight, but harder to get.
 Text Notes 1150 5200 0    60   ~ 0
@@
 Text Notes 7850 1550 0    60   ~ 0
 Mount the LM399 a *little* off the board,\nto keep stress away.\nSource: http://www.eevblog.com/forum/\nmetrology/ultra-precision-reference-ltz1000/\nmsg404500/#msg404500
+$Comp
+L Device:Q_PJFET_DSG Q?
+U 1 1 60A667B8
+P 4600 2450
+F 0 "Q?" H 4800 2500 50  0000 L CNN
+F 1 "J270" H 4800 2400 50  0000 L CNN
+F 2 "Package_TO_SOT_SMD:SOT-23" H 4800 2550 50  0001 C CNN
+F 3 "~" H 4600 2450 50  0001 C CNN
+F 4 "On Semiconductor" H 4600 2450 50  0001 C CNN "MFN"
+F 5 "MMBFJ270" H 4600 2450 50  0001 C CNN "PN"
+F 6 "On Semiconductor MMBFJ176" H 4600 2450 50  0001 C CNN "Alternative"
+	1    4600 2450
+	0    -1   -1   0
+$EndComp
+Text HLabel 3850 2350 0    60   UnSpc ~ 0
+V-
+Wire Wire Line
+	3850 2350 4000 2350
+Wire Wire Line
+	4800 2350 5100 2350
+Wire Wire Line
+	4450 2800 4600 2800
+Wire Wire Line
+	4600 2800 4600 2650
+$Comp
+L Device:R R?
+U 1 1 60A9337F
+P 4150 2350
+F 0 "R?" V 3943 2350 50  0000 C CNN
+F 1 "2k" V 4034 2350 50  0000 C CNN
+F 2 "Resistor_SMD:R_0603_1608Metric" V 4080 2350 50  0001 C CNN
+F 3 "" H 4150 2350 50  0001 C CNN
+F 4 "Vishay" H 4150 2350 60  0001 C CNN "MFN"
+F 5 "CRCW06032K00JNEA" H 4150 2350 50  0001 C CNN "PN"
+	1    4150 2350
+	0    1    1    0
+$EndComp
+Wire Wire Line
+	4300 2350 4400 2350
 $EndSCHEMATC

Commit message: Added part annotations
Parts:
- gave numbers to parts that had none: 2
Changed lines of the file:
@@
 Mount the LM399 a *little* off the board,\nto keep stress away.\nSource: http://www.eevblog.com/forum/\nmetrology/ultra-precision-reference-ltz1000/\nmsg404500/#msg404500
 $Comp
-L Device:Q_PJFET_DSG Q?
+L Device:Q_PJFET_DSG Q1
 U 1 1 60A667B8
 P 4600 2450
-F 0 "Q?" H 4800 2500 50  0000 L CNN
+F 0 "Q1" H 4800 2500 50  0000 L CNN
 F 1 "J270" H 4800 2400 50  0000 L CNN
 F 2 "Package_TO_SOT_SMD:SOT-23" H 4800 2550 50  0001 C CNN
@@
 	4600 2800 4600 2650
 $Comp
-L Device:R R?
+L Device:R R2
 U 1 1 60A9337F
 P 4150 2350
-F 0 "R?" V 3943 2350 50  0000 C CNN
+F 0 "R2" V 3943 2350 50  0000 C CNN
 F 1 "2k" V 4034 2350 50  0000 C CNN
 F 2 "Resistor_SMD:R_0603_1608Metric" V 4080 2350 50  0001 C CNN

Commit message: Fixed typo
Other:
- note added: "Startup circuit:\nIt does not cause zener shift\nwith different V_zener+.\nThe gate of the JFET is held\nat the positive supply of the zener.\nThe JFET will therefore conduct and\npull the negative leg of the zener down\nuntil its source (the negative leg of\nthe zener) is about 2 V to 4 V below the\nsupply. It will then turn off and leakage\nwill be on the order of a few pA.\nThe 2k resistor is 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"
- note removed: "Startup circuit:\nIt does not cause zener shift\nwith different V_zener+\nThe gate of the JFET is held\nat the positive supply of the zener.\nThe JFET will therefore conduct and\npull the negative leg of the zener down\nuntil the its source (the negative leg of\nthe zener) is abour 2 V to 4 V below the\nsupply. It will then turn off and leakage\nwill be on the order of a few pA.\nThe 2k resistor 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"
Changed lines of the file:
@@
 	3600 3050 3600 2000
 Text Notes 4100 1850 0    60   ~ 0
-Startup circuit:\nIt does not cause zener shift\nwith different V_zener+\nThe gate of the JFET is held\nat the positive supply of the zener.\nThe JFET will therefore conduct and\npull the negative leg of the zener down\nuntil the its source (the negative leg of\nthe zener) is abour 2 V to 4 V below the\nsupply. It will then turn off and leakage\nwill be on the order of a few pA.\nThe 2k resistor is for protection only.
+Startup circuit:\nIt does not cause zener shift\nwith different V_zener+.\nThe gate of the JFET is held\nat the positive supply of the zener.\nThe JFET will therefore conduct and\npull the negative leg of the zener down\nuntil its source (the negative leg of\nthe zener) is about 2 V to 4 V below the\nsupply. It will then turn off and leakage\nwill be on the order of a few pA.\nThe 2k resistor is for protection only.
 Text Notes 2350 950  0    60   ~ 0
 Use 1 oz./sqft of copper to\nminimize trace resistance and\ntherefore minimize succeptibility\nto temperature.
