File: reference_board.sch (KiCad schematic (older format))
At the start: 4 parts, among them J1 CONN_02X04, U1 TMP236

Commit message: Changed trace width to 0.25 mm to make it more robust Added bypass capacitor to the temperature sensor Rotated open source logo to fit it onto the board
Parts:
- added C4: 100n, Capacitor_SMD:C_0603_1608Metric, symbol Device:C
Connections:
- wire segments 43 -> 47
Changed lines of the file:
@@
 EESchema Schematic File Version 4
 LIBS:reference_board-cache
-EELAYER 26 0
+EELAYER 29 0
 EELAYER END
 $Descr A4 11693 8268
@@
 	2550 5050 2550 4950
 Wire Wire Line
-	2550 4350 2550 3750
+	2550 4350 2550 4250
 Wire Wire Line
 	2550 3750 2650 3750
@@
 L Mechanical:MountingHole H1
 U 1 1 5C37ECDE
-P 3150 3000
-F 0 "H1" H 3250 3050 50  0000 L CNN
-F 1 "MountingHole" H 3250 3000 50  0000 L CNN
-F 2 "MountingHole:MountingHole_2.7mm_M2.5_DIN965_Pad" H 3150 3000 50  0001 C CNN
-F 3 "~" H 3150 3000 50  0001 C CNN
-	1    3150 3000
-	1    0    0    -1
-$EndComp
+P 4150 5100
+F 0 "H1" H 4250 5150 50  0000 L CNN
+F 1 "MountingHole" H 4250 5100 50  0000 L CNN
+F 2 "MountingHole:MountingHole_2.7mm_M2.5_DIN965_Pad" H 4150 5100 50  0001 C CNN
+F 3 "~" H 4150 5100 50  0001 C CNN
+	1    4150 5100
+	1    0    0    -1
+$EndComp
+$Comp
+L Device:C C4
+U 1 1 5C6BB176
+P 1550 4650
+F 0 "C4" H 1700 4700 50  0000 L CNN
+F 1 "100n" H 1700 4600 50  0000 L CNN
+F 2 "Capacitor_SMD:C_0603_1608Metric" H 1588 4500 50  0001 C CNN
+F 3 "~" H 1550 4650 50  0001 C CNN
+F 4 "Murata" H 1550 4650 50  0001 C CNN "MFN"
+F 5 "GRM188R71H104KA93D" H 1550 4650 50  0001 C CNN "MFP"
+	1    1550 4650
+	1    0    0    -1
+$EndComp
+Wire Wire Line
+	1550 4500 1550 4250
+Wire Wire Line
+	1550 4250 2550 4250
+Connection ~ 2550 4250
+Wire Wire Line
+	2550 4250 2550 3750
+$Comp
+L power:GND #PWR0102
+U 1 1 5C6BC39A
+P 1550 5050
+F 0 "#PWR0102" H 1550 4800 50  0001 C CNN
+F 1 "GND" H 1555 4877 50  0000 C CNN
+F 2 "" H 1550 5050 50  0001 C CNN
+F 3 "" H 1550 5050 50  0001 C CNN
+	1    1550 5050
+	-1   0    0    -1
+$EndComp
+Wire Wire Line
+	1550 4800 1550 5050
 $EndSCHEMATC

Commit message: Updated resistor requirements (changed R1 from 5 ppm to 10 ppm) Rotated all text labels by 180° to match the main pcb Fixed soldermask to preventsolder from shorting rectangular pins to GND
Other:
- note added: "Use an RAF M2106-2545-AL, 11 mm M2.5 standoff\nto mount the reference daughter board onto the\nmain pcb."
Changed lines of the file:
@@
 Sheet 1 2
 Title "LM399 negative voltage reference"
-Date "2019-01-11"
-Rev "v3.1.0"
+Date "2019-06-28"
+Rev "v3.1.1"
 Comp ""
 Comment1 "Copyright (©) 2018, Patrick Baus <patrick.baus@physik.tu-darmstadt.de>"
@@
 Wire Wire Line
 	1550 4800 1550 5050
+Text Notes 4000 5500 0    60   ~ 0
+Use an RAF M2106-2545-AL, 11 mm M2.5 standoff\nto mount the reference daughter board onto the\nmain pcb.
 $EndSCHEMATC

Commit message: Removed via from bypass capacitor pad
Other:
- moved on the sheet: C4
Changed lines of the file:
@@
 EESchema Schematic File Version 4
 LIBS:reference_board-cache
-EELAYER 29 0
+EELAYER 30 0
 EELAYER END
 $Descr A4 11693 8268
@@
 P 2550 4650
 F 0 "U1" H 2200 4700 50  0000 R CNN
-F 1 "TMP236" H 2200 4650 50  0000 R CNN
+F 1 "TMP236" H 2200 4600 50  0000 R CNN
 F 2 "Package_TO_SOT_SMD:SOT-353_SC-70-5" H 2550 4250 50  0001 C CNN
 F 3 "http://www.ti.com/lit/ds/symlink/tmp235.pdf" H 2550 4650 50  0001 C CNN
@@
 L Device:C C4
 U 1 1 5C6BB176
-P 1550 4650
-F 0 "C4" H 1700 4700 50  0000 L CNN
-F 1 "100n" H 1700 4600 50  0000 L CNN
-F 2 "Capacitor_SMD:C_0603_1608Metric" H 1588 4500 50  0001 C CNN
-F 3 "~" H 1550 4650 50  0001 C CNN
-F 4 "Murata" H 1550 4650 50  0001 C CNN "MFN"
-F 5 "GRM188R71H104KA93D" H 1550 4650 50  0001 C CNN "MFP"
-	1    1550 4650
-	1    0    0    -1
-$EndComp
-Wire Wire Line
-	1550 4500 1550 4250
-Wire Wire Line
-	1550 4250 2550 4250
+P 1450 4650
+F 0 "C4" H 1600 4700 50  0000 L CNN
+F 1 "100n" H 1600 4600 50  0000 L CNN
+F 2 "Capacitor_SMD:C_0603_1608Metric" H 1488 4500 50  0001 C CNN
+F 3 "~" H 1450 4650 50  0001 C CNN
+F 4 "Murata" H 1450 4650 50  0001 C CNN "MFN"
+F 5 "GRM188R71H104KA93D" H 1450 4650 50  0001 C CNN "MFP"
+	1    1450 4650
+	1    0    0    -1
+$EndComp
+Wire Wire Line
+	1450 4500 1450 4250
+Wire Wire Line
+	1450 4250 2550 4250
 Connection ~ 2550 4250
 Wire Wire Line
@@
 L power:GND #PWR0102
 U 1 1 5C6BC39A
-P 1550 5050
-F 0 "#PWR0102" H 1550 4800 50  0001 C CNN
-F 1 "GND" H 1555 4877 50  0000 C CNN
-F 2 "" H 1550 5050 50  0001 C CNN
-F 3 "" H 1550 5050 50  0001 C CNN
-	1    1550 5050
-	-1   0    0    -1
-$EndComp
-Wire Wire Line
-	1550 4800 1550 5050
+P 1450 5050
+F 0 "#PWR0102" H 1450 4800 50  0001 C CNN
+F 1 "GND" H 1455 4877 50  0000 C CNN
+F 2 "" H 1450 5050 50  0001 C CNN
+F 3 "" H 1450 5050 50  0001 C CNN
+	1    1450 5050
+	-1   0    0    -1
+$EndComp
+Wire Wire Line
+	1450 4800 1450 5050
 Text Notes 4000 5500 0    60   ~ 0
 Use an RAF M2106-2545-AL, 11 mm M2.5 standoff\nto mount the reference daughter board onto the\nmain pcb.

Commit message: Changed op amp to LT1001 Added startup circuit Board shrink Changed temperature sensor to TI TMP236 Added mounting hole
Connections:
- net labels added: V3.3
Other:
- note removed: "3.3V"
Changed lines of the file:
@@
 Sheet 1 2
 Title "LM399 negative voltage reference"
-Date "2019-06-28"
-Rev "v3.1.1"
+Date "2019-11-20"
+Rev "v3.2.0"
 Comp ""
 Comment1 "Copyright (©) 2018, Patrick Baus <patrick.baus@physik.tu-darmstadt.de>"
@@
 Wire Wire Line
 	2650 3750 2750 3750
-Text Notes 2750 3100 0    60   ~ 0
-3.3V
 $Comp
 L Mechanical:MountingHole H1
@@
 P 4150 5100
 F 0 "H1" H 4250 5150 50  0000 L CNN
-F 1 "MountingHole" H 4250 5100 50  0000 L CNN
+F 1 "MountingHole" H 4250 5050 50  0000 L CNN
 F 2 "MountingHole:MountingHole_2.7mm_M2.5_DIN965_Pad" H 4150 5100 50  0001 C CNN
 F 3 "~" H 4150 5100 50  0001 C CNN
@@
 Text Notes 4000 5500 0    60   ~ 0
 Use an RAF M2106-2545-AL, 11 mm M2.5 standoff\nto mount the reference daughter board onto the\nmain pcb.
+Text Label 2050 4250 0    60   ~ 0
+V3.3
 $EndSCHEMATC
