File: reference_board.sch (KiCad schematic (older format))
At the start: 5 parts, among them J1 CONN_02X04, U1 TMP236

Commit message: Updated to v.3.2.1 -Changed D1 to a plastic package to eliminate possible light sensitivity -Updated bom.ini for the latest version of KiBOM -Updated symbol fields (changed MFP -> PN) for KiCost compatibility -Added PCBA config -Updated Gerber files
Parts:
- C4: MFP GRM188R71H104KA93D -> (none); PN (none) -> GRM188R71H104KA93D
- J1: MFP 87606-804LF -> (none); PN (none) -> 87606-804LF
- U1: MFP TMP236A2DCKT -> (none); PN (none) -> TMP236A2DCKT
Changed lines of the file:
@@
 Sheet 1 2
 Title "LM399 negative voltage reference"
-Date "2019-11-20"
-Rev "v3.2.0"
+Date "2020-02-06"
+Rev "v3.2.1"
 Comp ""
 Comment1 "Copyright (©) 2020, Patrick Baus <patrick.baus@physik.tu-darmstadt.de>"
@@
 F 3 "" H 2950 2350 50  0001 C CNN
 F 4 "Amphenol" H 2950 3550 50  0001 C CNN "MFN"
-F 5 "87606-804LF" H 2950 3550 50  0001 C CNN "MFP"
+F 5 "87606-804LF" H 2950 3550 50  0001 C CNN "PN"
 	1    2950 3550
 	1    0    0    -1
@@
 F 3 "http://www.ti.com/lit/ds/symlink/tmp235.pdf" H 2550 4650 50  0001 C CNN
 F 4 "Texas Instruments" H 2550 4650 50  0001 C CNN "MFN"
-F 5 "TMP236A2DCKT" H 2550 4650 50  0001 C CNN "MFP"
+F 5 "TMP236A2DCKT" H 2550 4650 50  0001 C CNN "PN"
 	1    2550 4650
 	1    0    0    -1
@@
 F 3 "~" H 1450 4650 50  0001 C CNN
 F 4 "Murata" H 1450 4650 50  0001 C CNN "MFN"
-F 5 "GRM188R71H104KA93D" H 1450 4650 50  0001 C CNN "MFP"
+F 5 "GRM188R71H104KA93D" H 1450 4650 50  0001 C CNN "PN"
 	1    1450 4650
 	1    0    0    -1
