File: LM399.kicad_sch (KiCad schematic)
At the start: 16 parts, among them U2 LM399, U3 LT1001

Commit message: Add PCBA variant
Parts:
- R2: Alternative Welwyn PCF0805-13-7K5-B-T1 -> Welwyn PCF0805-13-7K5-B-T1
- RN1, U2: variant (none) -> default
Changed lines of the file:
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@@
       (effects (font (size 1.27 1.27)) hide)
+    )
+    (property "variant" "default" (at 73.66 77.47 0)
+      (effects (font (size 1.524 1.524)) hide)
     )
     (property "Temperature" "Tstorage = -65 °C to 150 °C" (at 73.66 77.47 0)
@@
       (effects (font (size 1.27 1.27)) hide)
     )
-    (property "Alternative" " Welwyn PCF0805-13-7K5-B-T1" (at 151.13 59.69 90)
+    (property "Alternative" "Welwyn PCF0805-13-7K5-B-T1" (at 151.13 59.69 90)
       (effects (font (size 1.27 1.27)) hide)
     )
@@
       (effects (font (size 1.27 1.27)) hide)
     )
+    (property "variant" "default" (at 176.53 124.46 0)
+      (effects (font (size 1.524 1.524)) hide)
+    )
     (property "RoHS" "Yes" (at 176.53 124.46 0)
