File: LM399.kicad_sch (KiCad schematic)
At the start: 16 parts, among them U2 LM399, U3 LT1001

Commit message: Updated libraries
Parts:
- RN1: footprint Custom_footprints:Vishay_300144 -> Custom_footprints:R_Array_Box3_L7.5mm_W2.5mm_P2.54mm_Vishay_300144
Changed lines of the file:
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@@
       (effects (font (size 1.27 1.27)) (justify right))
     )
-    (property "Footprint" "Custom_footprints:Vishay_300144" (at 164.465 124.46 90)
+    (property "Footprint" "Custom_footprints:R_Array_Box3_L7.5mm_W2.5mm_P2.54mm_Vishay_300144" (at 164.465 124.46 90)
       (effects (font (size 1.27 1.27)) hide)
     )
