File: Zener.kicad_sch (KiCad schematic)
At the start: 16 parts, among them U2 LM399, U3 LT1001

Commit message: Replaced connector J1 with Molex SlimStack 53307-1071.
- Updated to KiCAD 10
- Changed BAS116 diode D1 footprint to SOD-123F due to availability of parts
- Added QED logo
- Removed most references to LM399. The ADR1399 is now the default. LM399 is mentioned as option.
- Added more details for different zener voltage configurations
- Added WEEE logo
- Fixed label on silkscreen refering to R1 instead of R2. It now reads 'R2: 10 ppm/K max.'
Parts:
- C2, C3: farnell# (none) -> 3228096
- C4, C5: farnell# (none) -> 2070398
- D1: footprint Diode_SMD:D_SOD-123 -> Diode_SMD:D_SOD-123F; PN BAS116GWJ -> BAS116H\,115
- U2: value LM399 -> ADR1399; Alternative (none) -> Analog Devices LM399AH#PBF; PN LM399AH#PBF -> ADR1399KHZ; Temperature Tstorage = -65 °C to 150 °C -> Top = 0 °C to 70 °C, Tstorage = -65 °C to 150 °C
- U3: farnell# (none) -> 4217953
Other:
- note added: "Mount the ADR1399 a *little* off the board, to keep stress away. Source: http://www.eevblog.com/forum/ metrology/ultra-precision-reference-ltz1000/ msg404500/#msg404500"
- note added: "The ADR1399 has a TCR of 0.2 ppm/K"
- note added: "The output drift with the zener current is about 0.15 ppm / ppm maximum. In order to meet the ADR1399 specs make sure the resistor has a maximum TCR of 10 ppm / K (results in 1.5 ppm / K)."
- note removed: "Mount the LM399 a *little* off the board, to keep stress away. Source: http://www.eevblog.com/forum/ metrology/ultra-precision-reference-ltz1000/ msg404500/#msg404500"
- note removed: "Output voltage Table: Voltage | R1 | RN1a | RN1b ----------------------- -10 V | 3k | 20k | 9k -15 V | 7.5k | 17k | 20k"
- note removed: "The LM399 has a TCR of 0.3 ppm/K"
- note removed: "The output drift with the zener current is about 0.15 ppm / ppm maximum. In order to meet the LM399 specs make sure the resistor has a maximum TCR of 10 ppm / K (results in 1.5 ppm / K)."
- company: (none) -> Quantum Electronic Devices GmbH
- title: LM399 negative voltage reference -> ADR1399 negative voltage reference
